File: hw/WiSer-TTL/WiSer-TTL.kicad_sch (KiCad schematic)
At the start: 60 parts, among them J1 USB_C_Receptacle_USB2.0, J2 Conn_01x02, J3 Conn_01x02, J4 Conn_01x02, J5 Conn_01x08, U1 USBLC6-2P6, U2 AP2112K-3.3TRG1, U3 ESP32-S2, Y1 40MHz

Commit message: Update hardware design files
Parts:
- removed C18: TBD, Capacitor_SMD:C_0402_1005Metric, symbol Device:C
- removed R10, R3, R5, R7, R8, R9: 22, Resistor_SMD:R_0402_1005Metric, symbol Device:R
- added C1, C24, C3: 0.1u, Capacitor_SMD:C_0402_1005Metric, symbol Device:C
- added C17, C19, C23: TBD, Capacitor_SMD:C_0402_1005Metric, symbol Device:C
- added D1, D10, D11, D12, D13, D14, D15: ESD9B5.0ST5G, Diode_SMD:D_SOD-923, symbol Diode:ESD9B5.0ST5G
- added D6: ESD9B3.3ST5G, Diode_SMD:D_SOD-923, symbol Diode:ESD9B3.3ST5G
- added L2: L_Ferrite_Coupled_Small_1243, DLM0NSM900HY2D:FIL_DLM0NSM900HY2D, symbol Device:L_Ferrite_Coupled_Small_1243
- added L3: TBD, Inductor_SMD:L_0402_1005Metric, symbol Device:L
- added L4: 24n, Inductor_SMD:L_0402_1005Metric, symbol Device:L
- added R1, R2: 330, Resistor_SMD:R_0402_1005Metric, symbol Device:R
- added U4: SN74LV6T17BQAR, SN74LV6T17BQAR:WQFN14_BQA_TEX, symbol SN74LV6T17BQAR:SN74LV6T17BQAR
- renumbered C8 to C10, C9 to C11, C10 to C12, C11 to C13, C12 to C14, C13 to C15, C14 to C16, C15 to C18, C1 to C2, C16 to C20, C17 to C21, C19 to C22, C2 to C4, C3 to C5, C4 to C6, C5 to C7, C6 to C8, C7 to C9, D1 to D2, D2 to D3, D3 to D4, D4 to D5, D5 to D7, D6 to D8, D7 to D9, L2 to L5, R14 to R10, R15 to R11, R1 to R3, R2 to R4, R4 to R5, R11 to R7, R12 to R8, R13 to R9
Connections:
- net +3V3: now also C24.1, U4.14 (VCC)
- net GND: now also R7.1, C1.2, C17.2, C19.2, C23.2, C24.2, C3.2, D1.1 (A1), D10.1 (A1), D11.1 (A1), D12.1 (A1), D13.1 (A1), D14.1 (A1), D15.1 (A1), D6.1 (A1), R1.2, R2.2, U4.7 (GND); no longer R7.2
- net LNA_IN: now also C23.1
- net UART_CTS: now also U3.39 (GPIO35), U4.8 (4Y); no longer J5.5 (Pin_5)
- net UART_DTR: now also U3.38 (GPIO34), U4.11 (5A); no longer J5.6 (Pin_6)
- net UART_RTS: now also U3.40 (GPIO36), U4.5 (3A); no longer J5.4 (Pin_4)
- net UART_RXD: now also U3.41 (GPIO37), U4.4 (2Y); no longer D7.1 (K), J5.3 (Pin_3)
- net UART_TXD: now also U3.42 (GPIO38), U4.1 (1A); no longer D8.1 (K), J5.2 (Pin_2)
- net USB+: now also L2.4; no longer U3.26 (GPIO20/ADC2_CH9/USB_D+)
- net USB-: now also L2.1; no longer U3.25 (GPIO19/ADC2_CH8/USB_D-)
- net XTAL_P: now also L4.2
- net at D2.2 (A), J2.2 (Pin_2), J3.1 (Pin_1): now also D1.2 (A2)
- net at D4.1 (K), J5.1 (Pin_1): now also D6.2 (A2)
- net at C21.1, L5.1: now also C19.1, L3.2; no longer E1.1
- net at D5.1 (K), J5.7 (Pin_7): now also D15.2 (A2)
- net at C20.1, Y1.1: now also L4.1
- net at J1.S1 (SHIELD): now also C1.1, C3.1, R1.1, R2.1
- new net: C17.1, E1.1, L3.1
- new net TTL_CTS: D13.2 (A2), J5.5 (Pin_5), R7.2, U4.9 (4A)
- new net TTL_DTR: D14.2 (A2), J5.6 (Pin_6), U4.10 (5Y)
- new net TTL_RTS: D12.2 (A2), J5.4 (Pin_4), U4.6 (3Y)
- new net TTL_RXD: D11.2 (A2), D7.1 (K), J5.3 (Pin_3), U4.3 (2A)
- new net TTL_TXD: D10.2 (A2), D8.1 (K), J5.2 (Pin_2), U4.2 (1Y)
- new net USB_FIL+: L2.3, U3.26 (GPIO20/ADC2_CH9/USB_D+)
- new net USB_FIL-: L2.2, U3.25 (GPIO19/ADC2_CH8/USB_D-)
Other:
- moved on the sheet: C21, D2, D4, D5, E1, J5, L5, R6, R7, R8, S1, U1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
