File: hw/WiSer-USB/WiSer-USB.kicad_sch (KiCad schematic)
At the start: 46 parts, among them P1 USB_C_Plug, U1 AP2112K-3.3TRG1, U2 USBLC6-2P6, U3 ESP32-S2, Y1 40MHz

Commit message: Update hardware design files
Parts:
- removed C18: TBD, Capacitor_SMD:C_0402_1005Metric, symbol Device:C
- added C1, C2: 0.1u, Capacitor_SMD:C_0402_1005Metric, symbol Device:C
- added C17, C19, C23: TBD, Capacitor_SMD:C_0402_1005Metric, symbol Device:C
- added L2: L_Ferrite_Coupled_Small_1243, DLM0NSM900HY2D:FIL_DLM0NSM900HY2D, symbol Device:L_Ferrite_Coupled_Small_1243
- added L3: TBD, Inductor_SMD:L_0402_1005Metric, symbol Device:L
- added L4: 24n, Inductor_SMD:L_0402_1005Metric, symbol Device:L
- added R1: 330, Resistor_SMD:R_0402_1005Metric, symbol Device:R
- R2: value 22 -> 330
- renumbered C8 to C10, C9 to C11, C10 to C12, C11 to C13, C12 to C14, C13 to C15, C14 to C16, C15 to C18, C16 to C20, C19 to C21, C17 to C22, C1 to C3, C2 to C4, C3 to C5, C4 to C6, C5 to C7, C6 to C8, C7 to C9, L2 to L5, R1 to R3, R3 to R4, R4 to R5, R8 to R6, R6 to R7, R7 to R8, R5 to R9, S2 to S1, S1 to S2
Connections:
- net GND: now also R2.2, C1.2, C17.2, C19.2, C2.2, C23.2, R1.2
- net LED_RXD: now also D2.1 (K); no longer D3.1 (K)
- net LED_TXD: now also D3.1 (K); no longer D2.1 (K)
- net LNA_IN: now also C23.1
- net USB+: now also L2.4; no longer U3.26 (GPIO20/ADC2_CH9/USB_D+)
- net USB-: now also L2.1; no longer U3.25 (GPIO19/ADC2_CH8/USB_D-)
- net XTAL_P: now also L4.2; no longer R2.2
- net at C22.1, L5.2: now also C19.1, L3.1; no longer E1.1
- net at C20.1, Y1.1: now also L4.1; no longer R2.1
- net at P1.S1 (SHIELD): now also R2.1, C1.1, C2.1, R1.1
- new net: C17.1, E1.1, L3.2
- new net USB_FIL+: L2.3, U3.26 (GPIO20/ADC2_CH9/USB_D+)
- new net USB_FIL-: L2.2, U3.25 (GPIO19/ADC2_CH8/USB_D-)
- no-connect marks 48 -> 47
Other:
- moved on the sheet: C22, D1, E1, FB1, L5, P1, R3, R6, R9, S1, S2, U2
